Commit message: Add masses + all components to the URDF, and a mass/torque report
Adds every component that actually rides on the robot (Pi, power bank,
both battery packs, PCA9685, L9110S, speakerphone, USB hub) with real
masses, plus inertial blocks on every existing link via new inertia
macros. mass_report.py then does forward kinematics over the tree and
reports total mass, centre of gravity, and whether the drivetrain has
torque margin.

The result reproduces the bench behaviour from part specs alone:

  TOTAL 2.01 kg, CoG x+0.003 z+0.115
  rolling    needs  4.8 mN-m/wheel, TT gives 7.8-11.8  -> margin x1.6-2.4
  BREAKAWAY  needs 19.3 mN-m/wheel, TT gives 7.8-11.8  -> margin x0.4-0.6

Rolling has margin, breakaway doesn't -- which is precisely what we saw:
he keeps going once moving but can't start from rest, jabbing helps, and
rock_test needed several tries. The model wasn't fitted to that symptom.

Notable finding: it is NOT mainly the arm. The whole arm is 525g (26%).
The power bank alone is 350g (17%), the single heaviest item. Power bank
+ speakerphone + servo battery = 750g (37%), all mounted high, which is
what puts the CoG 11.5cm up on a robot with 3.25cm wheels.

Masses are spec values not weighed, and the resistance coefficients are
estimates, so the exact crossover is soft -- but breakaway always runs
several times rolling, so the ordering is robust.

Co-Authored-By: Claude Opus 4.8 <noreply@anthropic.com>

File: ros2/melvinn_description/urdf/melvinn.urdf.xacro (robot description, xacro)
@@ -3,6 +3,7 @@
   MELVINN — URDF description for ROS 2.
   Models the real robot as built: a 4WD acrylic chassis carrying a 6-DOF
-  MG996R arm on a PCA9685, an HC-SR04 facing forward, and the IMX219 camera
-  riding on the wrist.
+  MG996R arm on a PCA9685, an HC-SR04 facing forward, the IMX219 camera on
+  the wrist, and all the electronics that actually ride along (Pi, two
+  battery packs, power bank, speakerphone, USB hub, motor driver).
   JOINT NAMES MATCH THE FIRMWARE. The six arm joints are named exactly as in
   ARM_JOINTS in robot_code/tests/assistant.py (base, shoulder, elbow, wrist,
@@ -14,20 +15,23 @@
   asymmetric where the centre isn't 90. Those centres were found on the real
   robot: the arm fouls the chassis at other values.
-  ⚠️ DIMENSIONS ARE ESTIMATES from typical part sizes — nothing in the repo
-  records measured lengths. Everything is a property at the top of this file,
-  so measuring the real robot and correcting them is a one-place edit.
+  MASSES exist so the model can answer "why won't it move" quantitatively —
+  total weight and centre of gravity. They're spec/typical values per part
+  (see the mass properties block). A URDF cannot model the *electrical* side
+  (battery sag under current), which bench testing suggests is the bigger
+  factor — see ros2/README.md.
+  ⚠️ DIMENSIONS AND COMPONENT PLACEMENT ARE ESTIMATES. Nothing in the repo
+  records measured lengths or where each board is bolted. Everything is a
+  property at the top of this file, so correcting them is a one-place edit.
 -->
 <robot name="melvinn" xmlns:xacro="http://www.ros.org/wiki/xacro">
+  <xacro:include filename="$(find melvinn_description)/urdf/inertia.xacro"/>
   <!-- ===================== dimensions (metres) ===================== -->
-  <!-- Chassis: typical 4WD acrylic plate -->
   <xacro:property name="chassis_len"   value="0.200"/>
   <xacro:property name="chassis_wid"   value="0.150"/>
   <xacro:property name="chassis_thick" value="0.005"/>
-  <!-- TT gearmotor wheels (the yellow ones) -->
   <xacro:property name="wheel_radius"  value="0.0325"/>
   <xacro:property name="wheel_width"   value="0.027"/>
-  <xacro:property name="wheel_x"       value="0.065"/>   <!-- from centre, fore/aft -->
-  <xacro:property name="wheel_y"       value="0.080"/>   <!-- from centre, left/right -->
-  <!-- Arm segment lengths -->
+  <xacro:property name="wheel_x"       value="0.065"/>
+  <xacro:property name="wheel_y"       value="0.080"/>
   <xacro:property name="arm_base_h"    value="0.050"/>
   <xacro:property name="upper_arm_len" value="0.100"/>
@@ -35,5 +39,38 @@
   <xacro:property name="wrist_len"     value="0.055"/>
   <xacro:property name="gripper_len"   value="0.080"/>
+  <xacro:property name="deck"  value="${chassis_thick/2}"/>   <!-- chassis top -->
+  <xacro:property name="deck2" value="0.055"/>                <!-- upper tier -->
   <xacro:property name="PI" value="3.14159265359"/>
+  <!-- ===================== mass properties (kg) =====================
+       Where these come from:
+         MG996R servo            0.055 each (datasheet)
+         Raspberry Pi 3A+        0.029      (spec)
+         TT gearmotor            0.030 each (typical) — carried on the wheel
+                                            link, since it sits at the wheel
+         Redmi 20000mAh bank     0.350      (typical for 20Ah)
+         Blomiky 6V 2200mAh NiMH 0.200      (typical 5-cell sub-C pack)
+         4x AA + holder          0.120
+         USB speakerphone        0.200
+         acrylic 4WD chassis     0.250      (both plates + standoffs)
+  -->
+  <xacro:property name="chassis_mass"  value="0.250"/>
+  <xacro:property name="wheel_mass"    value="0.065"/>  <!-- wheel + its TT motor -->
+  <xacro:property name="m_arm_base"    value="0.075"/>
+  <xacro:property name="m_shoulder"    value="0.075"/>
+  <xacro:property name="m_upper_arm"   value="0.090"/>
+  <xacro:property name="m_forearm"     value="0.075"/>
+  <xacro:property name="m_wrist"       value="0.070"/>
+  <xacro:property name="m_wrist_rot"   value="0.060"/>
+  <xacro:property name="m_gripper"     value="0.080"/>
+  <xacro:property name="m_pi"          value="0.029"/>
+  <xacro:property name="m_power_bank"  value="0.350"/>
+  <xacro:property name="m_drive_batt"  value="0.120"/>
+  <xacro:property name="m_servo_batt"  value="0.200"/>
+  <xacro:property name="m_pca9685"     value="0.010"/>
+  <xacro:property name="m_l9110s"      value="0.005"/>
+  <xacro:property name="m_speaker"     value="0.200"/>
+  <xacro:property name="m_usb_hub"     value="0.040"/>
+  <xacro:property name="m_ultrasonic"  value="0.010"/>
+  <xacro:property name="m_camera"      value="0.015"/>
   <!-- ===================== materials ===================== -->
   <material name="acrylic"><color rgba="0.85 0.85 0.90 0.55"/></material>
@@ -42,5 +79,6 @@
   <material name="blue">   <color rgba="0.15 0.35 0.85 1.0"/></material>
   <material name="green">  <color rgba="0.20 0.70 0.30 1.0"/></material>
-  <!-- Wheels are identical apart from placement -->
+  <material name="red">    <color rgba="0.80 0.15 0.15 1.0"/></material>
+  <material name="grey">   <color rgba="0.45 0.45 0.48 1.0"/></material>
   <xacro:macro name="wheel" params="name x y">
     <link name="wheel_${name}_link">
@@ -50,6 +88,9 @@
         <material name="yellow"/>
       </visual>
+      <xacro:cylinder_inertial mass="${wheel_mass}" radius="${wheel_radius}"
+                               length="${wheel_width}">
+        <origin rpy="${PI/2} 0 0"/>
+      </xacro:cylinder_inertial>
     </link>
-    <!-- continuous: wheels spin freely, no limit -->
     <joint name="wheel_${name}_joint" type="continuous">
       <parent link="base_link"/>
@@ -60,5 +101,4 @@
   </xacro:macro>
   <!-- ===================== chassis ===================== -->
-  <!-- base_footprint sits on the ground: the frame Nav2 drives around. -->
   <link name="base_footprint"/>
   <joint name="base_joint" type="fixed">
@@ -72,4 +112,8 @@
       <material name="acrylic"/>
     </visual>
+    <xacro:box_inertial mass="${chassis_mass}" x="${chassis_len}"
+                        y="${chassis_wid}" z="${chassis_thick}">
+      <origin xyz="0 0 0"/>
+    </xacro:box_inertial>
   </link>
   <xacro:wheel name="front_left"  x="${wheel_x}"  y="${wheel_y}"/>
@@ -77,6 +121,36 @@
   <xacro:wheel name="rear_left"   x="${-wheel_x}" y="${wheel_y}"/>
   <xacro:wheel name="rear_right"  x="${-wheel_x}" y="${-wheel_y}"/>
+  <!-- ===================== electronics + power =====================
+       Placement is approximate — see the warning at the top. What matters
+       for the mass question is that these are ON the robot and roughly
+       where they sit fore/aft and how high.
+  -->
+  <!-- AA pack slung under the chassis, as on the real bot -->
+  <xacro:payload name="drive_battery" parent="base_link" mass="${m_drive_batt}"
+                 x="0.060" y="0.055" z="0.030"
+                 px="-0.030" py="0" pz="-0.020" colour="red"/>
+  <xacro:payload name="pi" parent="base_link" mass="${m_pi}"
+                 x="0.065" y="0.030" z="0.012"
+                 px="-0.050" py="0.040" pz="${deck + 0.008}" colour="green"/>
+  <xacro:payload name="l9110s" parent="base_link" mass="${m_l9110s}"
+                 x="0.030" y="0.022" z="0.008"
+                 px="-0.070" py="-0.045" pz="${deck + 0.006}" colour="blue"/>
+  <xacro:payload name="pca9685" parent="base_link" mass="${m_pca9685}"
+                 x="0.062" y="0.026" z="0.008"
+                 px="0.010" py="-0.045" pz="${deck + 0.006}" colour="blue"/>
+  <xacro:payload name="usb_hub" parent="base_link" mass="${m_usb_hub}"
+                 x="0.070" y="0.028" z="0.012"
+                 px="-0.070" py="0" pz="${deck + 0.008}" colour="grey"/>
+  <!-- Heavy items ride on the upper tier — this is what lifts the CoG -->
+  <xacro:payload name="power_bank" parent="base_link" mass="${m_power_bank}"
+                 x="0.100" y="0.070" z="0.025"
+                 px="-0.030" py="0" pz="${deck2}" colour="black"/>
+  <xacro:payload name="servo_battery" parent="base_link" mass="${m_servo_batt}"
+                 x="0.075" y="0.045" z="0.028"
+                 px="0.030" py="0.040" pz="${deck2}" colour="green"/>
+  <xacro:payload name="speakerphone" parent="base_link" mass="${m_speaker}"
+                 x="0.090" y="0.090" z="0.030"
+                 px="-0.020" py="0" pz="${deck2 + 0.030}" colour="black"/>
   <!-- ===================== ultrasonic ===================== -->
-  <!-- HC-SR04, forward-facing. ros_bridge publishes sensor_msgs/Range here. -->
   <link name="ultrasonic_link">
     <visual>
@@ -84,4 +158,7 @@
       <material name="blue"/>
     </visual>
+    <xacro:box_inertial mass="${m_ultrasonic}" x="0.010" y="0.045" z="0.020">
+      <origin xyz="0 0 0"/>
+    </xacro:box_inertial>
   </link>
   <joint name="ultrasonic_joint" type="fixed">
@@ -91,5 +168,4 @@
   </joint>
   <!-- ===================== arm ===================== -->
-  <!-- Mounted toward the front of the plate, as on the real robot. -->
   <link name="arm_base_link">
     <visual>
@@ -98,9 +174,12 @@
       <material name="black"/>
     </visual>
+    <xacro:box_inertial mass="${m_arm_base}" x="0.055" y="0.055" z="${arm_base_h}">
+      <origin xyz="0 0 ${arm_base_h/2}"/>
+    </xacro:box_inertial>
   </link>
   <joint name="arm_mount_joint" type="fixed">
     <parent link="base_link"/>
     <child  link="arm_base_link"/>
-    <origin xyz="0.040 0 ${chassis_thick/2}"/>
+    <origin xyz="0.040 0 ${deck}"/>
   </joint>
   <!-- ch 0: base — yaw. Centre 90 deg, so +/- 90 deg of travel. -->
@@ -111,4 +190,7 @@
       <material name="black"/>
     </visual>
+    <xacro:box_inertial mass="${m_shoulder}" x="0.050" y="0.050" z="0.040">
+      <origin xyz="0 0 0.020"/>
+    </xacro:box_inertial>
   </link>
   <joint name="base" type="revolute">
@@ -127,4 +209,7 @@
       <material name="black"/>
     </visual>
+    <xacro:box_inertial mass="${m_upper_arm}" x="0.030" y="0.040" z="${upper_arm_len}">
+      <origin xyz="0 0 ${upper_arm_len/2}"/>
+    </xacro:box_inertial>
   </link>
   <joint name="shoulder" type="revolute">
@@ -142,4 +227,7 @@
       <material name="black"/>
     </visual>
+    <xacro:box_inertial mass="${m_forearm}" x="0.028" y="0.036" z="${forearm_len}">
+      <origin xyz="0 0 ${forearm_len/2}"/>
+    </xacro:box_inertial>
   </link>
   <joint name="elbow" type="revolute">
@@ -157,4 +245,7 @@
       <material name="black"/>
     </visual>
+    <xacro:box_inertial mass="${m_wrist}" x="0.026" y="0.032" z="${wrist_len}">
+      <origin xyz="0 0 ${wrist_len/2}"/>
+    </xacro:box_inertial>
   </link>
   <joint name="wrist" type="revolute">
@@ -173,4 +264,7 @@
       <material name="black"/>
     </visual>
+    <xacro:cylinder_inertial mass="${m_wrist_rot}" radius="0.018" length="0.030">
+      <origin xyz="0 0 0.015"/>
+    </xacro:cylinder_inertial>
   </link>
   <joint name="wrist_rotate" type="revolute">
@@ -181,6 +275,5 @@
     <limit lower="${-PI/2}" upper="${PI/2}" effort="10" velocity="1.0"/>
   </joint>
-  <!-- ch 5: gripper — the claw. One revolute joint stands in for the linkage;
-       real fingers are a mechanism driven by a single servo. -->
+  <!-- ch 5: gripper — the claw. -->
   <link name="gripper_link">
     <visual>
@@ -189,4 +282,7 @@
       <material name="green"/>
     </visual>
+    <xacro:box_inertial mass="${m_gripper}" x="0.020" y="0.060" z="${gripper_len}">
+      <origin xyz="0 0 ${gripper_len/2}"/>
+    </xacro:box_inertial>
   </link>
   <joint name="gripper" type="revolute">
@@ -198,7 +294,4 @@
   </joint>
   <!-- ===================== camera ===================== -->
-  <!-- IMX219 rides on the wrist, looking along the gripper. Mounted upside
-       down on the real robot (see FLIP_180 in the camera scripts) — that's a
-       driver-side fix, so this frame is the corrected, right-way-up view. -->
   <link name="camera_link">
     <visual>
@@ -206,4 +299,7 @@
       <material name="blue"/>
     </visual>
+    <xacro:box_inertial mass="${m_camera}" x="0.010" y="0.025" z="0.024">
+      <origin xyz="0 0 0"/>
+    </xacro:box_inertial>
   </link>
   <joint name="camera_joint" type="fixed">
@@ -212,5 +308,4 @@
     <origin xyz="0.025 0 0.020" rpy="0 0 0"/>
   </joint>
-  <!-- ROS camera convention: z forward, x right, y down -->
   <link name="camera_optical_frame"/>
   <joint name="camera_optical_joint" type="fixed">

Commit message: ROS model: JGA25 masses + torque, retire L9110S/TT references
URDF now models the installed drivetrain: wheel_mass 0.065 -> 0.135 kg
(65mm wheel + JGA25 gearmotor), the driver payload renamed l9110s ->
drivers at 2x BTS7960 mass (0.066 kg), and the mass/intro comments
updated. mass_report.py uses JGA25 stall torque (2-5 kg-cm) instead of
the TT figures and its narrative reflects that the robot now has
breakaway margin. ros2/README reframes the why-he-barely-moves section
as the historical TT diagnosis + the JGA25 fix. No l9110/TT_STALL refs
remain.

Co-Authored-By: Claude Opus 4.8 <noreply@anthropic.com>

File: ros2/melvinn_description/urdf/melvinn.urdf.xacro (robot description, xacro)
@@ -5,5 +5,5 @@
   MG996R arm on a PCA9685, an HC-SR04 facing forward, the IMX219 camera on
   the wrist, and all the electronics that actually ride along (Pi, two
-  battery packs, power bank, speakerphone, USB hub, motor driver).
+  battery packs, power bank, speakerphone, USB hub, two BTS7960 motor drivers).
   JOINT NAMES MATCH THE FIRMWARE. The six arm joints are named exactly as in
   ARM_JOINTS in robot_code/tests/assistant.py (base, shoulder, elbow, wrist,
@@ -46,6 +46,7 @@
          MG996R servo            0.055 each (datasheet)
          Raspberry Pi 3A+        0.029      (spec)
-         TT gearmotor            0.030 each (typical) — carried on the wheel
-                                            link, since it sits at the wheel
+         JGA25-370 gearmotor     0.100 each (metal-gear, installed Jul 2026) —
+                                            carried on the wheel link, since it
+                                            sits at the wheel
          Redmi 20000mAh bank     0.350      (typical for 20Ah)
          Blomiky 6V 2200mAh NiMH 0.200      (typical 5-cell sub-C pack)
@@ -53,7 +54,8 @@
          USB speakerphone        0.200
          acrylic 4WD chassis     0.250      (both plates + standoffs)
+         BTS7960 (IBT-2) driver  0.033 each (2 boards)
   -->
   <xacro:property name="chassis_mass"  value="0.250"/>
-  <xacro:property name="wheel_mass"    value="0.065"/>  <!-- wheel + its TT motor -->
+  <xacro:property name="wheel_mass"    value="0.135"/>  <!-- 65mm wheel + its JGA25 gearmotor -->
   <xacro:property name="m_arm_base"    value="0.075"/>
   <xacro:property name="m_shoulder"    value="0.075"/>
@@ -68,5 +70,5 @@
   <xacro:property name="m_servo_batt"  value="0.200"/>
   <xacro:property name="m_pca9685"     value="0.010"/>
-  <xacro:property name="m_l9110s"      value="0.005"/>
+  <xacro:property name="m_drivers"     value="0.066"/>  <!-- 2x BTS7960 (IBT-2) -->
   <xacro:property name="m_speaker"     value="0.200"/>
   <xacro:property name="m_usb_hub"     value="0.040"/>
@@ -133,6 +135,6 @@
                  x="0.065" y="0.030" z="0.012"
                  px="-0.050" py="0.040" pz="${deck + 0.008}" colour="green"/>
-  <xacro:payload name="l9110s" parent="base_link" mass="${m_l9110s}"
-                 x="0.030" y="0.022" z="0.008"
+  <xacro:payload name="drivers" parent="base_link" mass="${m_drivers}"
+                 x="0.050" y="0.050" z="0.010"
                  px="-0.070" py="-0.045" pz="${deck + 0.006}" colour="blue"/>
   <xacro:payload name="pca9685" parent="base_link" mass="${m_pca9685}"
